Commit message: work at cambridge

File: xacro/gummi_description_ee.urdf.xacro (robot description, xacro)
@@ -99,5 +99,5 @@
     <origin
       xyz="0.043506 -0.00023376 -0.019876"
-      rpy="0 0 0" />
+      rpy="-1.57079632679 0 0" />
     <parent
       link="lowerarm_preroll_d" />
@@ -105,5 +105,5 @@
       link="lowerarm" />
     <axis
-      xyz="-1 0 0" />
+      xyz="1 0 0" />
     <limit
       effort="0"
@@ -161,8 +161,8 @@
       link="wrist" />
     <axis
-      xyz="0 1 0" />
-    <limit
-      lower="-1"
-      upper="1"
+      xyz="0 -1 0" />
+    <limit
+      lower="-0.5"
+      upper="0.5"
       effort="0"
       velocity="0" />
